File: KiCad/projet_capteur_lebon - VERSION 3/projet_capteur_lebon V3.kicad_pcb (KiCad board)
At the start: 2 copper layers, 85.2 x 66 mm, 25 parts, among them J1 Power, J2 Digital/PWM, J3 Analog, J4 Digital/PWM

Commit message: fin V3
Parts:
- R6: footprint librairie_empreintes:R_Axial_DIN0207_L6.3mm_D2.5mm_P5.08mm_Vertical -> librairie_empreintes:R_Axial_DIN0207_L6.3mm_D2.5mm_P10.16mm_Horizontal
- moved R6 14.6 mm to (132.0, 78.4), turned to -90 degrees
- moved U7 13.2 mm to (131.5, 61.0)
- moved C4 5.70 mm to (132.5, 74.0), turned to 180 degrees
- moved R3 4.35 mm to (128.0, 83.3), turned to 90 degrees
Routing:
- net 5V: track 111.0 -> 233.3 mm
- net R2: track 0.00 -> 64.2 mm
- net /*11: track 0.00 -> 49.7 mm
- net Net-(U4-OUT): track 0.00 -> 31.8 mm
- net CAPT_AMPL: track 6.16 -> 28.6 mm
- net /13: track 0.00 -> 9.62 mm
- net /*10: track 0.00 -> 8.56 mm
- net (no net): track 0.00 -> 1.06 mm
- net GND: track 1.62 -> 0.89 mm
- added copper zone on B.Cu, net GND

Commit message: version finale validee par cathy qui sera imprimee
Parts:
- moved U1 3.50 mm to (177.5, 81.3)
- moved U9 1.57 mm to (142.5, 60.7)
Routing:
- net OUT_FLEX: track 12.6 -> 68.0 mm, vias 0 -> 1
- net 5V: track 233.3 -> 240.7 mm
- net SCL: track 21.4 -> 25.1 mm
- net SDA: track 19.7 -> 22.2 mm
- net RX: track 9.30 -> 10.5 mm
Other:
- board size 85.2 x 66 mm -> 88.8 x 69 mm
- board text added: "Clara et Anatolie"
