File: KiCad/projet_capteur_lebon - VERSION 3/projet_capteur_lebon V3.kicad_sch (KiCad schematic)
At the start: 21 parts, among them J1 Power, J2 Digital/PWM, J3 Analog, J4 Digital/PWM

Commit message: ajout readme et recup tests bench
Connections:
- net CAPT_AMPL: now also R6.1; no longer R6.2
- net at C4.2, R3.2, U4.6 (OUT): now also R6.2; no longer R6.1
Other:
- moved on the sheet: C1, C2, C4, R3, R5, R6
